File: headphones.sch (KiCad schematic (older format))
At the start: 20 parts

Commit message: ..
Parts:
- removed C? (x2): 0.1uF, symbol Device:C
- removed C?: 10uF, symbol Device:C
- removed C? (x3): 3.3uF, symbol Device:C
- removed C? (x2): 2.7nF, symbol Device:C
- removed C? (x4): 1uF, symbol Device:C
- removed J?: Headphones, symbol Connector:AudioJack3
- removed R? (x2): 470, symbol Device:R
- removed R? (x2): 10k, symbol Device:R
- removed R?: 82k, symbol Device:R
- removed U?: CS4344, Package_SO:TSSOP-10_3x3mm_P0.5mm, symbol audio_digital:CS4344
- removed U?: TPA6139A2, Package_SO:TSSOP-14_4.4x5mm_P0.65mm, symbol audio-amplifier:TPA6139A2
Connections:
- net labels removed: +3.3VA, GND, i2s_lrck, i2s_mck, i2s_sck, i2s_sdin, ~mute~
- wire segments 56 -> 0
Other:
- note removed: "Output Amplifier"
- note removed: "Stereo DAC"
