File: audio_input.sch (KiCad schematic (older format))
At the start: 47 parts

Commit message: Mostly done with schematic
Parts:
- C1, C10, C11, C12, C16, C18, C2, C3, C4, C9: renamed from C?; footprint (none) -> Capacitor_SMD:C_0603_1608Metric
- C13, C14, C15, C17, C5, C6, C7, C8: renamed from C?; footprint (none) -> Capacitor_SMD:C_0402_1005Metric
- J1, J2: renamed from J?; footprint (none) -> Connector_PinHeader_1.00mm:PinHeader_1x02_P1.00mm_Vertical
- R1, R10, R11, R12, R13, R14, R15, R16, R17, R18, R2, R3, R4, R5, R6, R7, R8, R9: renamed from R?; footprint (none) -> Resistor_SMD:R_0402_1005Metric
- R20, R21, R22, R23: footprint (none) -> Resistor_SMD:R_0402_1005Metric
- RV1, RV2: renamed from RV?; footprint (none) -> Potentiometer_SMD:Potentiometer_Bourns_3214J_Horizontal
- gave numbers to parts that had none: 3
Connections:
- net labels added: adc_sdo, sdo
- net labels removed: adc_sdout, sdout
