File: audio_output.sch (KiCad schematic (older format))
At the start: 29 parts

Commit message: ..
Connections:
- net labels added: +3.3V
- net labels removed: +3.3VA
Changed lines of the file:
@@
-$EndComp
-$Comp
-L power:+3.3VA #PWR?
-U 1 1 5FF79233
-P 3600 2750
-AR Path="/5FF79233" Ref="#PWR?"  Part="1"
-AR Path="/5FA600F4/5FF79233" Ref="#PWR?"  Part="1"
-AR Path="/5FEFCD68/5FF79233" Ref="#PWR?"  Part="1"
-AR Path="/5FEEB7ED/5FF79233" Ref="#PWR?"  Part="1"
-F 0 "#PWR?" H 3600 2600 50  0001 C CNN
-F 1 "+3.3VA" H 3615 2923 50  0000 C CNN
-F 2 "" H 3600 2750 50  0001 C CNN
-F 3 "" H 3600 2750 50  0001 C CNN
-	1    3600 2750
-	1    0    0    -1
 $EndComp
 $Comp
@@
 Wire Wire Line
 	4050 2250 4050 2350
-$Comp
-L power:+3.3VA #PWR?
-U 1 1 5FF79262
-P 4050 1850
-AR Path="/5FF79262" Ref="#PWR?"  Part="1"
-AR Path="/5FA600F4/5FF79262" Ref="#PWR?"  Part="1"
-AR Path="/5FEFCD68/5FF79262" Ref="#PWR?"  Part="1"
-AR Path="/5FEEB7ED/5FF79262" Ref="#PWR?"  Part="1"
-F 0 "#PWR?" H 4050 1700 50  0001 C CNN
-F 1 "+3.3VA" V 4050 2100 50  0000 C CNN
-F 2 "" H 4050 1850 50  0001 C CNN
-F 3 "" H 4050 1850 50  0001 C CNN
-	1    4050 1850
-	1    0    0    -1
-$EndComp
 Wire Wire Line
 	4050 1850 4050 1950
-$Comp
-L power:+3.3VA #PWR?
-U 1 1 5FF79269
-P 4250 1850
-AR Path="/5FA600F4/5FF79269" Ref="#PWR?"  Part="1"
-AR Path="/5FF79269" Ref="#PWR?"  Part="1"
-AR Path="/5FEFCD68/5FF79269" Ref="#PWR?"  Part="1"
-AR Path="/5FEEB7ED/5FF79269" Ref="#PWR?"  Part="1"
-F 0 "#PWR?" H 4250 1700 50  0001 C CNN
-F 1 "+3.3VA" V 4250 2100 50  0000 C CNN
-F 2 "" H 4250 1850 50  0001 C CNN
-F 3 "" H 4250 1850 50  0001 C CNN
-	1    4250 1850
-	1    0    0    -1
-$EndComp
 Wire Wire Line
 	4250 1850 4250 1950
@@
 Wire Wire Line
 	7300 4050 7300 3950
-$Comp
-L power:+3.3VA #PWR?
-U 1 1 5FF79312
-P 7250 2650
-AR Path="/5FF79312" Ref="#PWR?"  Part="1"
-AR Path="/5FA600F4/5FF79312" Ref="#PWR?"  Part="1"
-AR Path="/5FEFCD68/5FF79312" Ref="#PWR?"  Part="1"
-AR Path="/5FEEB7ED/5FF79312" Ref="#PWR?"  Part="1"
-F 0 "#PWR?" H 7250 2500 50  0001 C CNN
-F 1 "+3.3VA" V 7250 2900 50  0000 C CNN
-F 2 "" H 7250 2650 50  0001 C CNN
-F 3 "" H 7250 2650 50  0001 C CNN
-	1    7250 2650
-	1    0    0    -1
-$EndComp
 Wire Wire Line
 	7250 2650 7250 2750
@@
 	1    0    0    -1
 $EndComp
-$Comp
-L power:+3.3VA #PWR?
-U 1 1 5FF7932E
-P 6950 1900
-AR Path="/5FF7932E" Ref="#PWR?"  Part="1"
-AR Path="/5FA600F4/5FF7932E" Ref="#PWR?"  Part="1"
-AR Path="/5FEFCD68/5FF7932E" Ref="#PWR?"  Part="1"
-AR Path="/5FEEB7ED/5FF7932E" Ref="#PWR?"  Part="1"
-F 0 "#PWR?" H 6950 1750 50  0001 C CNN
-F 1 "+3.3VA" V 6950 2150 50  0000 C CNN
-F 2 "" H 6950 1900 50  0001 C CNN
-F 3 "" H 6950 1900 50  0001 C CNN
-	1    6950 1900
-	1    0    0    -1
-$EndComp
 Wire Wire Line
 	6950 1900 6950 2000
@@
 Wire Wire Line
 	5700 6050 5900 6050
+$Comp
+L power:+3.3V #PWR?
+U 1 1 60DF0530
+P 3600 2750
+F 0 "#PWR?" H 3600 2600 50  0001 C CNN
+F 1 "+3.3V" H 3615 2923 50  0000 C CNN
+F 2 "" H 3600 2750 50  0001 C CNN
+F 3 "" H 3600 2750 50  0001 C CNN
+	1    3600 2750
+	1    0    0    -1
+$EndComp
+$Comp
+L power:+3.3V #PWR?
+U 1 1 60DF10AA
+P 4050 1850
+F 0 "#PWR?" H 4050 1700 50  0001 C CNN
+F 1 "+3.3V" H 4065 2023 50  0000 C CNN
+F 2 "" H 4050 1850 50  0001 C CNN
+F 3 "" H 4050 1850 50  0001 C CNN
+	1    4050 1850
+	1    0    0    -1
+$EndComp
+$Comp
+L power:+3.3V #PWR?
+U 1 1 60DF1987
+P 4250 1850
+F 0 "#PWR?" H 4250 1700 50  0001 C CNN
+F 1 "+3.3V" H 4265 2023 50  0000 C CNN
+F 2 "" H 4250 1850 50  0001 C CNN
+F 3 "" H 4250 1850 50  0001 C CNN
+	1    4250 1850
+	1    0    0    -1
+$EndComp
+$Comp
+L power:+3.3V #PWR?
+U 1 1 60DF46C6
+P 6950 1900
+F 0 "#PWR?" H 6950 1750 50  0001 C CNN
+F 1 "+3.3V" H 6965 2073 50  0000 C CNN
+F 2 "" H 6950 1900 50  0001 C CNN
+F 3 "" H 6950 1900 50  0001 C CNN
+	1    6950 1900
+	1    0    0    -1
+$EndComp
+$Comp
+L power:+3.3V #PWR?
+U 1 1 60DF4F42
+P 7250 2650
+F 0 "#PWR?" H 7250 2500 50  0001 C CNN
+F 1 "+3.3V" H 7265 2823 50  0000 C CNN
+F 2 "" H 7250 2650 50  0001 C CNN
+F 3 "" H 7250 2650 50  0001 C CNN
+	1    7250 2650
+	1    0    0    -1
+$EndComp
 $EndSCHEMATC

Commit message: Mostly done with schematic
Parts:
- removed JP? (x2): Jumper_3_Open, symbol Jumper:Jumper_3_Open
- C19, C20, C26, C27: renamed from C?; footprint (none) -> Capacitor_SMD:C_0402_1005Metric
- C21, C23, C24, C25, C28, C29, C30: renamed from C?; footprint (none) -> Capacitor_SMD:C_0603_1608Metric
- C22: renamed from C?; footprint (none) -> Capacitor_SMD:C_0805_2012Metric
- J3, J4: renamed from J?; footprint (none) -> Connector_PinHeader_1.00mm:PinHeader_1x02_P1.00mm_Vertical
- J5: renamed from J?; footprint (none) -> Connector_Audio:Jack_3.5mm_CUI_SJ-3523-SMT_Horizontal
- JP1, JP2: renamed from JP?; footprint (none) -> Jumper:SolderJumper-3_P2.0mm_Open_TrianglePad1.0x1.5mm_NumberLabels
- R19, R24, R25, R26, R27, R28, R29: renamed from R?; footprint (none) -> Resistor_SMD:R_0402_1005Metric
- RV3: renamed from RV?; footprint (none) -> Potentiometer_SMD:Potentiometer_Bourns_3214J_Horizontal
- gave numbers to parts that had none: 2
Connections:
- net labels added: dac_sdi, i2s_sdi
- net labels removed: dac_sdin, i2s_sdin
- wire segments 89 -> 83
