File: power.sch (KiCad schematic (older format))
At the start: 13 parts

Commit message: ..
Parts:
- removed C?: 100uF, symbol Device:CP
- removed D? (x2): D_Schottky, symbol Device:D_Schottky
- added C?: 47uF, symbol Device:C
- added C? (x2): 22uF, symbol Device:C
- added C?: 470nF, symbol Device:C
- added C? (x3): 10uF, symbol Device:C
- added C?: 2.2nF, symbol Device:C
- added C?: C, symbol Device:C
- added C? (x2): 1uF, symbol Device:C
- added C?: 150uF, symbol Device:CP
- added FB?: 10nH, symbol Device:Ferrite_Bead
- added JP?: buck out jmp, symbol Jumper:Jumper_2_Bridged
- added L?: 1.1uH, symbol Device:L
- added Q?: MMBT3904, Package_TO_SOT_SMD:SOT-23, symbol Transistor_BJT:MMBT3904
- added R? (x3): R, symbol Device:R
- added R? (x2): 100k, symbol Device:R
- added U?: TPS62912, qfn:VQFN-HR-10, symbol power-reg:TPS62912
- added U?: TPS2069D, Package_TO_SOT_SMD:SOT-23-5, symbol power-switch:TPS2069D
Connections:
- net labels added: +5V, arty_pwr, buck_o, buck_pwr, cmod_pwr, ext_pg, usb_pwr
- net labels removed: +3.3VA, CMOD_PWR, usb_+5V
- wire segments 44 -> 121
- no-connect marks 1 -> 2
Other:
- note added: "CMOD A7 needs this diode if you connect to the cmod usb."
- note added: "Clean supply powers psoc, analog io, dac, and adc.\n Low current, low-noise, LDO\nDigital supply powers fpga"
- note added: "Drop external DC input down to 5V"
- note added: "Power Sources:\n\nMust allow all sources to be connected at the same time without damaging anything.\n\n+5V FPGA USB. During fpga development, this will probably be the only supply connected.\n\n+5V PSoC USB. When using the usb audio stream.\n\nExternal DC. 5V-9V input. I'm using a rectifier here since polarity standards are different between the fpga and audio world. This way it's plug and play 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"
- moved on the sheet: C?, FB?, R?

Commit message: Mostly done with schematic
Parts:
- removed C?: 47uF, symbol Device:C
- removed C?: 10uF, symbol Device:C
- removed C?: 150uF, symbol Device:CP
- removed JP?: buck out jmp, symbol Jumper:Jumper_2_Bridged
- added C32: 0.1uF, Capacitor_SMD:C_0402_1005Metric, symbol Device:C
- added C40: 22uF, Capacitor_SMD:C_0805_2012Metric, symbol Device:C
- added C42, C44: 22uF, Capacitor_SMD:C_1206_3216Metric, symbol Device:C
- added JP5: spread_jmp, Jumper:SolderJumper-2_P1.3mm_Open_TrianglePad1.0x1.5mm, symbol Jumper:Jumper_2_Open
- C31, C34, C35, C36, C41, C43: renamed from C?; footprint (none) -> Capacitor_SMD:C_0603_1608Metric
- C33, C39: renamed from C?; footprint (none) -> Capacitor_SMD:C_0402_1005Metric
- C37, C38: renamed from C?; footprint (none) -> Capacitor_SMD:C_0805_2012Metric
- C45, C46: renamed from C?; footprint (none) -> Capacitor_SMD:C_1206_3216Metric
- C47: renamed from C?; value C -> 1uF; footprint (none) -> Capacitor_SMD:C_0603_1608Metric
- D1: renamed from D?; footprint (none) -> Diode_SMD:D_SOD-323
- FB1, FB2: renamed from FB?; footprint (none) -> Inductor_SMD:L_0603_1608Metric
- J6: renamed from J?; footprint (none) -> Connector_BarrelJack:BarrelJack_CLIFF_FC681465S_SMT_Horizontal
- L1: renamed from L?; value 1.1uH -> 2.2uH
- R30, R31, R32, R34: renamed from R?; footprint (none) -> Resistor_SMD:R_0402_1005Metric
- R33: renamed from R?; value R -> 6.04k; footprint (none) -> Resistor_SMD:R_0402_1005Metric
- R35: renamed from R?; value R -> 25.5k; footprint (none) -> Resistor_SMD:R_0402_1005Metric
- R36: renamed from R?; value R -> 4.87k; footprint (none) -> Resistor_SMD:R_0402_1005Metric
- gave numbers to parts that had none: 4
Connections:
- net labels added: VO
- net labels removed: buck_o, buck_pwr
- wire segments 121 -> 131
Other:
- note added: "2.2MHz"
- note added: "USB Power is disabled when the external supply is connected"
- moved on the sheet: C31, C36, C45, C46, C47, FB2, R35, R36
