File: usb_interface.sch (KiCad schematic (older format))
At the start: 16 parts

Commit message: ..
Parts:
- added C?: 10nF, symbol Device:C
- added C? (x2): 15pF, symbol Device:C
- added C?: 100uF, symbol Device:CP
- added J?: USB_B_Mini, symbol Connector:USB_B_Mini
- added J?: Conn_02x05_Odd_Even, symbol Connector_Generic:Conn_02x05_Odd_Even
- added R? (x2): 27, symbol Device:R
- added R?: 4.7k, symbol Device:R
- added R?: 10k, symbol Device:R
- added R?: 100k, symbol Device:R
Connections:
- net labels added: ain0, ain1, ain2, ain3, fpga_10, fpga_8, fpga_9, psoc_lrclk, psoc_mclk, psoc_sclk, psoc_sdin, psoc_sdout, tck.sck, tdi, tdo.swv, tms.sdio, usb_+5V, vusb_mon
- net labels removed: led0, led1, led2, led3, swdck, swdio
- wire segments 95 -> 144
- no-connect marks 1 -> 2
Other:
- note added: "Optional grounding methods"
- note added: "Self-powered"

Commit message: ..
Parts:
- removed C?: 100uF, symbol Device:CP
- removed R?: 4.7k, symbol Device:R
- removed R?: 10k, symbol Device:R
- added C?: 0.1uF, symbol Device:C
- added FB?: ?, symbol Device:Ferrite_Bead
Connections:
- net labels added: usb_pwr
- net labels removed: usb_+5V
- wire segments 144 -> 140
Changed lines of the file:
@@
 $Descr USLetter 11000 8500
 encoding utf-8
-Sheet 2 6
+Sheet 5 6
 Title ""
 Date ""
@@
 Wire Wire Line
 	2400 1750 1800 1750
-Wire Wire Line
-	1800 1450 1900 1450
 $Comp
 L power:GND #PWR?
@@
 $Comp
 L Device:R R?
-U 1 1 5FEF6211
-P 2150 1450
-AR Path="/5FA355D9/5FEF6211" Ref="R?"  Part="1"
-AR Path="/5FEF6211" Ref="R?"  Part="1"
-AR Path="/5FA60E20/5FEF6211" Ref="R?"  Part="1"
-F 0 "R?" V 2050 1450 50  0000 C CNN
-F 1 "4.7k" V 2150 1450 50  0000 C CNN
-F 2 "" V 2080 1450 50  0001 C CNN
-F 3 "~" H 2150 1450 50  0001 C CNN
-	1    2150 1450
-	0    1    1    0
-$EndComp
-$Comp
-L Device:R R?
-U 1 1 5FEF6217
-P 2400 1200
-AR Path="/5FA355D9/5FEF6217" Ref="R?"  Part="1"
-AR Path="/5FEF6217" Ref="R?"  Part="1"
-AR Path="/5FA60E20/5FEF6217" Ref="R?"  Part="1"
-F 0 "R?" H 2330 1154 50  0000 R CNN
-F 1 "10k" V 2400 1250 50  0000 R CNN
-F 2 "" V 2330 1200 50  0001 C CNN
-F 3 "~" H 2400 1200 50  0001 C CNN
-	1    2400 1200
-	-1   0    0    1
-$EndComp
-Wire Wire Line
-	2300 1450 2400 1450
-Wire Wire Line
-	2400 1450 2400 1350
-$Comp
-L power:GND #PWR?
-U 1 1 5FEF621F
-P 2400 950
-AR Path="/5ED36906/5FEF621F" Ref="#PWR?"  Part="1"
-AR Path="/5FEF621F" Ref="#PWR?"  Part="1"
-AR Path="/5FA355D9/5FEF621F" Ref="#PWR?"  Part="1"
-AR Path="/5FA60E20/5FEF621F" Ref="#PWR?"  Part="1"
-F 0 "#PWR?" H 2400 700 50  0001 C CNN
-F 1 "GND" H 2405 777 50  0000 C CNN
-F 2 "" H 2400 950 50  0001 C CNN
-F 3 "" H 2400 950 50  0001 C CNN
-	1    2400 950
-	-1   0    0    1
-$EndComp
-Wire Wire Line
-	2400 950  2400 1050
-$Comp
-L Device:R R?
 U 1 1 5FEF6226
 P 1150 2150
@@
 Wire Wire Line
 	900  2350 1000 2350
-Text Label 2800 1450 2    50   ~ 0
-vusb_mon
-Wire Wire Line
-	2800 1450 2400 1450
-Connection ~ 2400 1450
 Text Notes 1300 1100 0    50   ~ 0
 Self-powered
@@
 Wire Wire Line
 	3000 1150 3000 1250
-Text GLabel 1900 1350 1    50   Input ~ 0
-usb_+5V
-Wire Wire Line
-	1900 1350 1900 1450
-Connection ~ 1900 1450
-Wire Wire Line
-	1900 1450 2000 1450
-$Comp
-L Device:CP C?
-U 1 1 5FEF626B
-P 950 1250
-AR Path="/5FA60E20/5FEF626B" Ref="C?"  Part="1"
-AR Path="/5FEF626B" Ref="C?"  Part="1"
-AR Path="/5FA355D9/5FEF626B" Ref="C?"  Part="1"
-F 0 "C?" H 950 1350 50  0000 L CNN
-F 1 "100uF" H 950 1150 50  0000 L CNN
-F 2 "" H 988 1100 50  0001 C CNN
-F 3 "~" H 950 1250 50  0001 C CNN
-	1    950  1250
-	1    0    0    -1
-$EndComp
-Text GLabel 950  1000 1    50   Input ~ 0
-usb_+5V
-Wire Wire Line
-	950  1000 950  1100
-$Comp
-L power:GND #PWR?
-U 1 1 5FEF6273
-P 950 1500
-AR Path="/5ED36906/5FEF6273" Ref="#PWR?"  Part="1"
-AR Path="/5FEF6273" Ref="#PWR?"  Part="1"
-AR Path="/5FA355D9/5FEF6273" Ref="#PWR?"  Part="1"
-AR Path="/5FA60E20/5FEF6273" Ref="#PWR?"  Part="1"
-F 0 "#PWR?" H 950 1250 50  0001 C CNN
-F 1 "GND" H 955 1327 50  0000 C CNN
-F 2 "" H 950 1500 50  0001 C CNN
-F 3 "" H 950 1500 50  0001 C CNN
-	1    950  1500
-	1    0    0    -1
-$EndComp
-Wire Wire Line
-	950  1500 950  1400
-Text Label 5550 5800 1    50   ~ 0
-vusb_mon
 Wire Wire Line
 	5550 5800 5550 5500
@@
 Wire Wire Line
 	6750 5600 6750 5500
+Wire Wire Line
+	1800 1450 2000 1450
+Text HLabel 5550 5800 3    50   Input ~ 0
+vusb_mon
+Text HLabel 2550 1450 2    50   Output ~ 0
+usb_pwr
+$Comp
+L Device:C C?
+U 1 1 60D492F1
+P 2000 1200
+AR Path="/5FA355D9/60D492F1" Ref="C?"  Part="1"
+AR Path="/60D492F1" Ref="C?"  Part="1"
+AR Path="/5FA60E20/60D492F1" Ref="C?"  Part="1"
+F 0 "C?" H 2000 1300 50  0000 L CNN
+F 1 "0.1uF" H 2000 1100 50  0000 L CNN
+F 2 "" H 2038 1050 50  0001 C CNN
+F 3 "~" H 2000 1200 50  0001 C CNN
+	1    2000 1200
+	1    0    0    -1
+$EndComp
+Wire Wire Line
+	2000 1350 2000 1450
+$Comp
+L power:GND #PWR?
+U 1 1 60D5037C
+P 2000 950
+AR Path="/5ED36906/60D5037C" Ref="#PWR?"  Part="1"
+AR Path="/60D5037C" Ref="#PWR?"  Part="1"
+AR Path="/5FA355D9/60D5037C" Ref="#PWR?"  Part="1"
+AR Path="/5FA60E20/60D5037C" Ref="#PWR?"  Part="1"
+F 0 "#PWR?" H 2000 700 50  0001 C CNN
+F 1 "GND" H 2005 777 50  0000 C CNN
+F 2 "" H 2000 950 50  0001 C CNN
+F 3 "" H 2000 950 50  0001 C CNN
+	1    2000 950
+	-1   0    0    1
+$EndComp
+Wire Wire Line
+	2000 1050 2000 950
+$Comp
+L Device:Ferrite_Bead FB?
+U 1 1 60D6EB60
+P 2300 1450
+F 0 "FB?" V 2200 1600 50  0000 C CNN
+F 1 "?" V 2117 1450 50  0000 C CNN
+F 2 "" V 2230 1450 50  0001 C CNN
+F 3 "~" H 2300 1450 50  0001 C CNN
+	1    2300 1450
+	0    1    1    0
+$EndComp
+Wire Wire Line
+	2150 1450 2000 1450
+Connection ~ 2000 1450
+Wire Wire Line
+	2550 1450 2450 1450
 $EndSCHEMATC

Commit message: Mostly done with schematic
Parts:
- removed C?: 15pF, symbol Device:C
- removed Y?: 12MHz, symbol Device:Crystal_GND24
- added R40, R41: R, Resistor_SMD:R_0402_1005Metric, symbol Device:R
- added X1: ECS-TXO-3225-122.8, Oscillator:Oscillator_SMD_EuroQuartz_XO32-4Pin_3.2x2.5mm, symbol Oscillator:XO32
- C48, C49, C50, C51, C57, C58, C59, C60, C61, C62, C63: renamed from C?; footprint (none) -> Capacitor_SMD:C_0402_1005Metric
- C52: renamed from C?; value 15pF -> 0.1uF; footprint (none) -> Capacitor_SMD:C_0402_1005Metric
- C53, C54, C55, C56: renamed from C?; footprint (none) -> Capacitor_SMD:C_0603_1608Metric
- FB3: renamed from FB?; footprint (none) -> Inductor_SMD:L_0603_1608Metric
- J16: renamed from J?; footprint (none) -> Connector_USB:USB_Mini-B_Wuerth_65100516121_Horizontal
- R39, R42, R43: renamed from R?; footprint (none) -> Resistor_SMD:R_0402_1005Metric
- gave numbers to parts that had none: 3
Connections:
- net labels added: psoc_sdi, psoc_sdo, psocgp0, psocgp1, psocgp2, psocgp3, psocgp4, psocgp5, psocgp6, psocgp7, psocgp[0..7], vusb
- net labels removed: ain0, ain1, ain2, ain3, fpga0, fpga1, fpga2, fpga3, fpga4, fpga5, fpga6, fpga7, fpga_10, fpga_8, fpga_9, psoc_sdin, psoc_sdout, xo
- wire segments 140 -> 144
- no-connect marks 2 -> 30
Other:
- note added: "12.288MHz"
- note removed: "Does it matter?"
- moved on the sheet: C49, C52, FB3
