File: usb_interface.sch (KiCad schematic (older format))
At the start: 27 parts

Commit message: ..
Parts:
- removed C? (x2): 15pF, symbol Device:C
- removed Y?: 12MHz, symbol Device:Crystal_GND24
- added C?: 0.1uF, symbol Device:C
- added X?: 12.288 MHz, Oscillator:Oscillator_SMD_Abracon_ASCO-4Pin_1.6x1.2mm, symbol Oscillator:ASCO
Connections:
- net labels added: audio_clk, audio_clk_en, lrclk, mclk, sclk, sdi, sdo
- net labels removed: ain0, ain1, ain2, ain3, fpga0, fpga1, fpga2, fpga3, fpga4, fpga5, fpga6, fpga7, fpga_10, fpga_9, psoc_lrclk, psoc_mclk, psoc_sclk, psoc_sdin, psoc_sdout, xi, xo
- wire segments 144 -> 129
- no-connect marks 2 -> 3
Other:
- note removed: "Does it matter?"
