File: fpga.sch (KiCad schematic (older format))
At the start: 1 part

Commit message: Mostly done with schematic
Parts:
- added J10, J11, J8, J9: Enc, Connector_PinHeader_1.00mm:PinHeader_1x03_P1.00mm_Vertical, symbol Connector_Generic:Conn_01x03
- added J12, J13, J14, J15: Sw, Connector_PinHeader_1.00mm:PinHeader_1x02_P1.00mm_Vertical, symbol Connector_Generic:Conn_01x02
- added J7: MIDI, Connector_Audio:Jack_3.5mm_CUI_SJ-3523-SMT_Horizontal, symbol Connector:AudioJack3
- added R37: 220, Resistor_SMD:R_0402_1005Metric, symbol Device:R
- added R38: 280, Resistor_SMD:R_0402_1005Metric, symbol Device:R
- added U9: H11L1, Package_DIP:SMDIP-6_W9.53mm, symbol Isolator:H11L1
- gave numbers to parts that had none: 1
Connections:
- net labels added: +3.3V, adc_lrclk, adc_mclk, adc_sclk, adc_sdo, cmod_vu, dac_lrclk, dac_mclk, dac_sclk, dac_sdi, enc0_a, enc0_b, enc1_a, enc1_b, enc2_a, enc2_b, enc3_a, enc3_b, midi_tx, psoc_lrclk, psoc_mclk, psoc_sclk, psoc_sdi, psoc_sdo, psocgp0, psocgp1, psocgp2, psocgp3, psocgp4, psocgp5, psocgp6, psocgp7, psocgp[0..7], sw0, sw1, sw2, sw3, ~mute~
- net labels removed: adc_m0, adc_m1, i2s_lrck2, i2s_lrck3, i2s_mck2, i2s_sck2, i2s_sck3, i2s_sd2, i2s_sd3
- wire segments 10 -> 78
- no-connect marks 0 -> 12
Other:
- note added: "Master audio clock."
- note added: "Rotary Encoder Inputs"

Commit message: ..
Parts:
- added J? (x4): LED, symbol Connector_Generic:Conn_01x02
- added R? (x4): R, symbol Device:R
Connections:
- net labels added: led0, led1, led2, led3
- wire segments 78 -> 94
- no-connect marks 12 -> 8
Changed lines of the file:
@@
 NoConn ~ 6200 4550
 NoConn ~ 6200 4650
-NoConn ~ 6200 4750
-NoConn ~ 6200 4850
-NoConn ~ 6200 4950
-NoConn ~ 6200 5050
 NoConn ~ 4400 4350
 NoConn ~ 4400 4250
@@
 Text Label 4100 3550 0    50   ~ 0
 psocgp7
+Text Label 7550 4750 2    50   ~ 0
+led0
+$Comp
+L Device:R R?
+U 1 1 613FDC12
+P 6450 4750
+F 0 "R?" V 6400 4900 50  0000 C CNN
+F 1 "R" V 6450 4750 50  0000 C CNN
+F 2 "" V 6380 4750 50  0001 C CNN
+F 3 "~" H 6450 4750 50  0001 C CNN
+	1    6450 4750
+	0    1    1    0
+$EndComp
+$Comp
+L Device:R R?
+U 1 1 613FDDF1
+P 6700 4850
+F 0 "R?" V 6650 5000 50  0000 C CNN
+F 1 "R" V 6700 4850 50  0000 C CNN
+F 2 "" V 6630 4850 50  0001 C CNN
+F 3 "~" H 6700 4850 50  0001 C CNN
+	1    6700 4850
+	0    1    1    0
+$EndComp
+$Comp
+L Device:R R?
+U 1 1 613FE1F0
+P 6950 4950
+F 0 "R?" V 6900 5100 50  0000 C CNN
+F 1 "R" V 6950 4950 50  0000 C CNN
+F 2 "" V 6880 4950 50  0001 C CNN
+F 3 "~" H 6950 4950 50  0001 C CNN
+	1    6950 4950
+	0    1    1    0
+$EndComp
+$Comp
+L Device:R R?
+U 1 1 613FE6A8
+P 7200 5050
+F 0 "R?" V 7150 5200 50  0000 C CNN
+F 1 "R" V 7200 5050 50  0000 C CNN
+F 2 "" V 7130 5050 50  0001 C CNN
+F 3 "~" H 7200 5050 50  0001 C CNN
+	1    7200 5050
+	0    1    1    0
+$EndComp
+Wire Wire Line
+	6200 4750 6300 4750
+Wire Wire Line
+	6200 4850 6550 4850
+Wire Wire Line
+	6800 4950 6200 4950
+Wire Wire Line
+	6200 5050 7050 5050
+Wire Wire Line
+	7550 4750 6600 4750
+Text Label 7550 4850 2    50   ~ 0
+led1
+Text Label 7550 4950 2    50   ~ 0
+led2
+Text Label 7550 5050 2    50   ~ 0
+led3
+Wire Wire Line
+	7550 5050 7350 5050
+Wire Wire Line
+	7550 4950 7100 4950
+Wire Wire Line
+	6850 4850 7550 4850
+$Comp
+L Connector_Generic:Conn_01x02 J?
+U 1 1 61423155
+P 5350 750
+F 0 "J?" H 5430 742 50  0000 L CNN
+F 1 "LED" H 5430 651 50  0000 L CNN
+F 2 "" H 5350 750 50  0001 C CNN
+F 3 "~" H 5350 750 50  0001 C CNN
+	1    5350 750
+	1    0    0    -1
+$EndComp
+Text Label 4950 750  0    50   ~ 0
+led0
+$Comp
+L power:GND #PWR?
+U 1 1 61429691
+P 5050 850
+AR Path="/5ED36906/61429691" Ref="#PWR?"  Part="1"
+AR Path="/61429691" Ref="#PWR?"  Part="1"
+AR Path="/5FA28C16/61429691" Ref="#PWR?"  Part="1"
+AR Path="/6042C0C1/61429691" Ref="#PWR?"  Part="1"
+F 0 "#PWR?" H 5050 600 50  0001 C CNN
+F 1 "GND" V 5055 722 50  0000 R CNN
+F 2 "" H 5050 850 50  0001 C CNN
+F 3 "" H 5050 850 50  0001 C CNN
+	1    5050 850
+	0    1    1    0
+$EndComp
+Wire Wire Line
+	4950 750  5150 750
+Wire Wire Line
+	5050 850  5150 850
+$Comp
+L Connector_Generic:Conn_01x02 J?
+U 1 1 61431A7F
+P 5350 1100
+F 0 "J?" H 5430 1092 50  0000 L CNN
+F 1 "LED" H 5430 1001 50  0000 L CNN
+F 2 "" H 5350 1100 50  0001 C CNN
+F 3 "~" H 5350 1100 50  0001 C CNN
+	1    5350 1100
+	1    0    0    -1
+$EndComp
+Text Label 4950 1100 0    50   ~ 0
+led1
+$Comp
+L power:GND #PWR?
+U 1 1 61431A86
+P 5050 1200
+AR Path="/5ED36906/61431A86" Ref="#PWR?"  Part="1"
+AR Path="/61431A86" Ref="#PWR?"  Part="1"
+AR Path="/5FA28C16/61431A86" Ref="#PWR?"  Part="1"
+AR Path="/6042C0C1/61431A86" Ref="#PWR?"  Part="1"
+F 0 "#PWR?" H 5050 950 50  0001 C CNN
+F 1 "GND" V 5055 1072 50  0000 R CNN
+F 2 "" H 5050 1200 50  0001 C CNN
+F 3 "" H 5050 1200 50  0001 C CNN
+	1    5050 1200
+	0    1    1    0
+$EndComp
+Wire Wire Line
+	4950 1100 5150 1100
+Wire Wire Line
+	5050 1200 5150 1200
+$Comp
+L Connector_Generic:Conn_01x02 J?
+U 1 1 61435F5A
+P 5350 1450
+F 0 "J?" H 5430 1442 50  0000 L CNN
+F 1 "LED" H 5430 1351 50  0000 L CNN
+F 2 "" H 5350 1450 50  0001 C CNN
+F 3 "~" H 5350 1450 50  0001 C CNN
+	1    5350 1450
+	1    0    0    -1
+$EndComp
+Text Label 4950 1450 0    50   ~ 0
+led2
+$Comp
+L power:GND #PWR?
+U 1 1 61435F61
+P 5050 1550
+AR Path="/5ED36906/61435F61" Ref="#PWR?"  Part="1"
+AR Path="/61435F61" Ref="#PWR?"  Part="1"
+AR Path="/5FA28C16/61435F61" Ref="#PWR?"  Part="1"
+AR Path="/6042C0C1/61435F61" Ref="#PWR?"  Part="1"
+F 0 "#PWR?" H 5050 1300 50  0001 C CNN
+F 1 "GND" V 5055 1422 50  0000 R CNN
+F 2 "" H 5050 1550 50  0001 C CNN
+F 3 "" H 5050 1550 50  0001 C CNN
+	1    5050 1550
+	0    1    1    0
+$EndComp
+Wire Wire Line
+	4950 1450 5150 1450
+Wire Wire Line
+	5050 1550 5150 1550
+$Comp
+L Connector_Generic:Conn_01x02 J?
+U 1 1 6143A3A8
+P 5350 1800
+F 0 "J?" H 5430 1792 50  0000 L CNN
+F 1 "LED" H 5430 1701 50  0000 L CNN
+F 2 "" H 5350 1800 50  0001 C CNN
+F 3 "~" H 5350 1800 50  0001 C CNN
+	1    5350 1800
+	1    0    0    -1
+$EndComp
+Text Label 4950 1800 0    50   ~ 0
+led3
+$Comp
+L power:GND #PWR?
+U 1 1 6143A3AF
+P 5050 1900
+AR Path="/5ED36906/6143A3AF" Ref="#PWR?"  Part="1"
+AR Path="/6143A3AF" Ref="#PWR?"  Part="1"
+AR Path="/5FA28C16/6143A3AF" Ref="#PWR?"  Part="1"
+AR Path="/6042C0C1/6143A3AF" Ref="#PWR?"  Part="1"
+F 0 "#PWR?" H 5050 1650 50  0001 C CNN
+F 1 "GND" V 5055 1772 50  0000 R CNN
+F 2 "" H 5050 1900 50  0001 C CNN
+F 3 "" H 5050 1900 50  0001 C CNN
+	1    5050 1900
+	0    1    1    0
+$EndComp
+Wire Wire Line
+	4950 1800 5150 1800
+Wire Wire Line
+	5050 1900 5150 1900
 Wire Bus Line
 	1500 2650 1500 3500
