File: fpga.sch (KiCad schematic (older format))
At the start: 1 part

Commit message: ..
Connections:
- net labels added: ai_lrclk, ai_mclk, ai_sclk, ai_sdi, ao_lrclk, ao_mclk, ao_sclk, ao_sdo, hp_lrclk, hp_mclk, hp_sclk, hp_sdo, psoc_lrclk, psoc_mclk, psoc_sclk, psoc_sdi, psoc_sdo
- net labels removed: i2s_lrck2, i2s_mck2, i2s_sck2, i2s_sd2
- wire segments 10 -> 23
Other:
- note added: "Clock Capable Pins (PIO):\nSRCC: 38, 37, 47, 48, 5, 8\nMRCC: 36, 40, 46, 43, 3, 18, 19\nWhich should I prefer? No idea...\nI think SRCC probably is better for this application because\nthe audio clock section of this design should be pretty small and contained."
Changed lines of the file:
@@
 $Descr USLetter 11000 8500
 encoding utf-8
-Sheet 6 6
+Sheet 5 6
 Title ""
 Date ""
@@
 	1    0    0    -1
 $EndComp
-Text Label 6600 3150 2    50   ~ 0
-i2s_mck2
-Text Label 6600 3050 2    50   ~ 0
-i2s_lrck2
-Text Label 6600 2950 2    50   ~ 0
-i2s_sck2
-Text Label 6600 2850 2    50   ~ 0
-i2s_sd2
-Wire Wire Line
-	6600 2850 6200 2850
-Wire Wire Line
-	6200 2950 6600 2950
-Wire Wire Line
-	6600 3050 6200 3050
-Wire Wire Line
-	6200 3150 6600 3150
 $Comp
 L power:GND #PWR?
@@
 Wire Wire Line
 	6200 4750 6600 4750
+Text HLabel 4300 3250 0    50   Input ~ 0
+psoc_mclk
+Text HLabel 4300 2850 0    50   Input ~ 0
+psoc_sclk
+Text HLabel 4300 2950 0    50   Input ~ 0
+psoc_lrclk
+Text HLabel 4300 3050 0    50   Input ~ 0
+psoc_sdo
+Text HLabel 4300 3150 0    50   Output ~ 0
+psoc_sdi
+Wire Wire Line
+	4300 3150 4400 3150
+Wire Wire Line
+	4400 3050 4300 3050
+Wire Wire Line
+	4300 2950 4400 2950
+Wire Wire Line
+	4400 2850 4300 2850
+Wire Wire Line
+	4300 3250 4400 3250
+Text HLabel 4300 3550 0    50   Output ~ 0
+hp_mclk
+Text HLabel 4300 3650 0    50   Output ~ 0
+hp_sclk
+Text HLabel 4300 3750 0    50   Output ~ 0
+hp_lrclk
+Text HLabel 4300 3850 0    50   Output ~ 0
+hp_sdo
+Wire Wire Line
+	4400 3850 4300 3850
+Wire Wire Line
+	4300 3750 4400 3750
+Wire Wire Line
+	4400 3650 4300 3650
+Wire Wire Line
+	4300 3550 4400 3550
+Text HLabel 6300 3850 2    50   Output ~ 0
+ai_mclk
+Text HLabel 6300 2950 2    50   Output ~ 0
+ai_sclk
+Text HLabel 6300 3050 2    50   Output ~ 0
+ai_lrclk
+Text HLabel 6300 2850 2    50   Output ~ 0
+ao_mclk
+Text HLabel 6300 3150 2    50   Input ~ 0
+ai_sdi
+Text HLabel 6300 3950 2    50   Output ~ 0
+ao_sclk
+Text HLabel 6300 4050 2    50   Output ~ 0
+ao_lrclk
+Text HLabel 6300 4150 2    50   Output ~ 0
+ao_sdo
+Text Notes 2550 2250 0    50   ~ 0
+Clock Capable Pins (PIO):\nSRCC: 38, 37, 47, 48, 5, 8\nMRCC: 36, 40, 46, 43, 3, 18, 19\nWhich should I prefer? No idea...\nI think SRCC probably is better for this application because\nthe audio clock section of this design should be pretty small and contained.
+Wire Wire Line
+	6300 2850 6200 2850
+Wire Wire Line
+	6200 2950 6300 2950
+Wire Wire Line
+	6300 3050 6200 3050
+Wire Wire Line
+	6200 3150 6300 3150
+Wire Wire Line
+	6300 3850 6200 3850
+Wire Wire Line
+	6200 3950 6300 3950
+Wire Wire Line
+	6300 4050 6200 4050
+Wire Wire Line
+	6200 4150 6300 4150
 $EndSCHEMATC
